File: TT_0.4_Control_board!/_autosave-TT_0.4_Control_board!.kicad_sch (KiCad schematic)
At the start: 46 parts, among them J1 Conn_01x03_Socket, J10 T4, J11 T5, J12 J_Th, J13 J_Th, J14 J_Th, J15 J_Th, J16 J_BMS_17, J17 J_BMS_23, J18 JST_S_Kill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

Commit message: PCB Update
Parts:
- R10, R3, R4, R5, R8, R9: value R -> 0R
- R11: value 440R -> 400R
- R6, R7: value R -> 68R
Connections:
- net LED1: now also R3.2
- net LED2: now also R4.2
- net LED3: now also R5.2
- net LED4: now also R6.2
- net LED5: now also R7.2
- net LED6: now also R8.2
- net LED7: now also R9.2
- net LED8: now also R10.2
Other:
- moved on the sheet: D1, D2, D3, D4, D5, D6, D7, D8, R10, R3, R4, R5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
